Commit message: Update robot_core.xacro

File: description/robot_core.xacro (robot description, xacro)
@@ -51,5 +51,5 @@
         <parent link="base_link"/>
         <child link="left_wheel"/>
-        <origin xyz="0 0.101 0" rpy="-${pi/2} 0 0" />
+        <origin xyz="0 0.107 0" rpy="-${pi/2} 0 0" />
         <axis xyz="0 0 1"/>
     </joint>
@@ -77,5 +77,5 @@
         <parent link="base_link"/>
         <child link="right_wheel"/>
-        <origin xyz="0 -0.101 0" rpy="${pi/2} 0 0" />
+        <origin xyz="0 -0.107 0" rpy="${pi/2} 0 0" />
         <axis xyz="0 0 -1"/>
     </joint>
