Commit message: adding gazebo_control

File: description/gazebo_control.xacro (robot description, xacro)
@@ -6,6 +6,6 @@
             <left_joint>left_wheel_joint</left_joint>
             <right_joint>right_wheel_joint</right_joint>
-            <wheel_separation>0.75</wheel_separation>
-            <wheel_diameter>0.2</wheel_diameter>
+            <wheel_separation>0.7</wheel_separation>
+            <wheel_diameter>0.1</wheel_diameter>
             <!-- Limits -->
             <max_wheel_torque>200</max_wheel_torque>

File: description/robot.urdf.xacro (robot description, xacro)
@@ -2,6 +2,6 @@
 <robot xmlns:xacro="http://www.ros.org/wiki/xacro"  name="robot">
     <xacro:include filename="robot_core.xacro" />
-    <!-- <xacro:include filename="gazebo_control.xacro" /> -->
-    <xacro:include filename="ros2_control.xacro" />
+    <xacro:include filename="gazebo_control.xacro" />
+    <!--<xacro:include filename="ros2_control.xacro" /> -->
     <!-- xacro:include filename="lidar.xacro" /> -->
     <!-- <xacro:include filename="camera.xacro" /> -->

File: description/robot_core.xacro (robot description, xacro)
@@ -41,4 +41,7 @@
       </xacro:inertial_cylinder>
     </link>
+    <gazebo reference="chassis">
+      <material>Gazebo/Blue</material>
+    </gazebo>
     <!-- LEFT WHEEL -->
     <joint name="left_wheel_joint" type="continuous">
@@ -64,4 +67,7 @@
       </xacro:inertial_cylinder>
     </link>
+    <gazebo reference="left_wheel">
+      <material>Gazebo/Black</material>
+    </gazebo>
     <!-- RIGHT WHEEL -->
     <joint name="right_wheel_joint" type="continuous">
@@ -87,4 +93,7 @@
       </xacro:inertial_cylinder>
     </link>
+    <gazebo reference="right_wheel">
+      <material>Gazebo/Black</material>
+    </gazebo>
     <!-- CASTER WHEEL 1-->
     <joint name ="caster_wheel_1_joint" type="fixed">
@@ -96,5 +105,5 @@
       <visual>
         <geometry>
-          <sphere radius="0.04"/>
+          <sphere radius="0.05"/>
         </geometry>
         <material name="orange"/>
@@ -102,5 +111,5 @@
       <collision>
         <geometry>
-          <sphere radius="0.04"/>
+          <sphere radius="0.05"/>
         </geometry>
       </collision>
@@ -109,4 +118,9 @@
       </xacro:inertial_sphere>
     </link>
+    <gazebo reference="caster_wheel_1">
+      <material>Gazebo/Orange</material>
+      <mu1 value="0.001"/>
+      <mu2 value="0.002"/>
+    </gazebo>
     <!-- CASTER WHEEL 2-->
     <joint name ="caster_wheel_2_joint" type="fixed">
@@ -118,5 +132,5 @@
       <visual>
         <geometry>
-          <sphere radius="0.04"/>
+          <sphere radius="0.05"/>
         </geometry>
         <material name="orange"/>
@@ -124,5 +138,5 @@
       <collision>
         <geometry>
-          <sphere radius="0.04"/>
+          <sphere radius="0.05"/>
         </geometry>
       </collision>
@@ -131,3 +145,8 @@
       </xacro:inertial_sphere>
     </link>
+    <gazebo reference="caster_wheel_2">
+      <material>Gazebo/Orange</material>
+      <mu1 value="0.001"/>
+      <mu2 value="0.001"/>
+    </gazebo>
 </robot>

Commit message: adding SLAM toolbox

File: description/gazebo_control.xacro (robot description, xacro)
@@ -6,6 +6,6 @@
             <left_joint>left_wheel_joint</left_joint>
             <right_joint>right_wheel_joint</right_joint>
-            <wheel_separation>0.35</wheel_separation>
-            <wheel_diameter>0.1</wheel_diameter>
+            <wheel_separation>0.214</wheel_separation>
+            <wheel_diameter>0.066</wheel_diameter>
             <!-- Limits -->
             <max_wheel_torque>200</max_wheel_torque>

File: description/robot.urdf.xacro (robot description, xacro)
@@ -2,5 +2,5 @@
 <robot xmlns:xacro="http://www.ros.org/wiki/xacro"  name="robot">
     <xacro:arg name="use_ros2_control" default="true"/>
-    <xacro:arg name="sim_mode" default="false"/>
+    <xacro:arg name="sim_mode" default="true"/>
     <xacro:include filename="robot_core.xacro" />
     <xacro:if value="$(arg use_ros2_control)">
@@ -11,5 +11,5 @@
     </xacro:unless>
     <xacro:include filename="lidar.xacro" />
-    <xacro:include filename="camera.xacro" />
+    <!--<xacro:include filename="camera.xacro" /> -->
     <!-- <xacro:include filename="depth_camera.xacro" /> -->
 </robot>

File: description/robot_core.xacro (robot description, xacro)
@@ -2,4 +2,18 @@
 <robot xmlns:xacro="http://www.ros.org/wiki/xacro" >
     <xacro:include filename="inertial_macros.xacro"/>
+    <xacro:property name="chassis_length" value="0.246"/>
+    <xacro:property name="chassis_width" value="0.176"/>
+    <xacro:property name="chassis_height" value="0.073"/>
+    <xacro:property name="chassis_mass" value="1.0"/>
+    <xacro:property name="wheel_radius" value="0.033"/>
+    <xacro:property name="wheel_thickness" value="0.026"/>
+    <xacro:property name="wheel_mass" value="0.05"/>
+    <xacro:property name="wheel_offset_x" value="0.05"/>
+    <xacro:property name="wheel_offset_y" value="0.107"/>
+    <xacro:property name="wheel_offset_z" value="0.01"/>
+    <xacro:property name="caster_wheel_radius" value="0.01"/>
+    <xacro:property name="caster_wheel_mass" value="0.01"/>
+    <xacro:property name="caster_wheel_offset_x" value="0.16"/>
+    <xacro:property name="caster_wheel_offset_z" value="${wheel_offset_z - wheel_radius + caster_wheel_radius}"/>
     <material name="white">
         <color rgba="1 1 1 1" />
@@ -20,30 +34,38 @@
     <link name="base_link">
     </link>
+    <!-- BASE_FOOTPRINT LINK -->
+    <joint name="base_footprint_joint" type="fixed">
+        <parent link="base_link"/>
+        <child link="base_footprint"/>
+        <origin xyz="0 0 0" rpy="0 0 0"/>
+    </joint>
+    <link name="base_footprint">
+    </link>
     <!-- CHASSIS LINK -->
     <joint name="chassis_joint" type="fixed">
         <parent link="base_link"/>
         <child link="chassis"/>
-        <origin xyz="-0.1 0 0"/>
+        <origin xyz="${-wheel_offset_x} 0 ${-wheel_offset_z}"/>
     </joint>
     <link name="chassis">
         <visual>
-            <origin xyz="0.123 0 0.0365"/>
+            <origin xyz="${chassis_length/2} 0 ${chassis_height/2}"/>
             <geometry>
-                <box size="0.246 0.176 0.073"/>
+                <box size="${chassis_length} ${chassis_width} ${chassis_height}"/>
             </geometry>
-            <material name="black"/>
+            <material name="orange"/>
         </visual>
         <collision>
-            <origin xyz="0.123 0 0.0365"/>
+            <origin xyz="${chassis_length/2} 0 ${chassis_height/2}"/>
             <geometry>
-                <box size="0.246 0.176 0.073"/>
+                <box size="${chassis_length} ${chassis_width} ${chassis_height}"/>
             </geometry>
         </collision>
-        <xacro:inertial_box mass="0.5" x="0.246" y="0.176" z="0.073">
-            <origin xyz="0.123 0 0.0365" rpy="0 0 0"/>
+        <xacro:inertial_box mass="0.5" x="${chassis_length}" y="${chassis_width}" z="${chassis_height}">
+            <origin xyz="${chassis_length/2} 0 ${chassis_height/2}" rpy="0 0 0"/>
         </xacro:inertial_box>
     </link>
     <gazebo reference="chassis">
-        <material>Gazebo/Black</material>
+        <material>Gazebo/Orange</material>
     </gazebo>
     <!-- LEFT WHEEL LINK -->
@@ -51,5 +73,5 @@
         <parent link="base_link"/>
         <child link="left_wheel"/>
-        <origin xyz="0 0.101 0" rpy="-${pi/2} 0 0" />
+        <origin xyz="0 ${wheel_offset_y} 0" rpy="-${pi/2} 0 0" />
         <axis xyz="0 0 1"/>
     </joint>
@@ -57,5 +79,5 @@
         <visual>
             <geometry>
-                <cylinder radius="0.033" length="0.026"/>
+                <cylinder radius="${wheel_radius}" length="${wheel_thickness}"/>
             </geometry>
             <material name="blue"/>
@@ -63,8 +85,8 @@
         <collision>
             <geometry>
-                <sphere radius="0.033"/>
+                <sphere radius="${wheel_radius}"/>
             </geometry>
         </collision>
-        <xacro:inertial_cylinder mass="0.1" length="0.026" radius="0.033">
+        <xacro:inertial_cylinder mass="${wheel_mass}" length="${wheel_thickness}" radius="${wheel_radius}">
             <origin xyz="0 0 0" rpy="0 0 0"/>
         </xacro:inertial_cylinder>
@@ -77,5 +99,5 @@
         <parent link="base_link"/>
         <child link="right_wheel"/>
-        <origin xyz="0 -0.101 0" rpy="${pi/2} 0 0" />
+        <origin xyz="0 ${-wheel_offset_y} 0" rpy="${pi/2} 0 0" />
         <axis xyz="0 0 -1"/>
     </joint>
@@ -83,5 +105,5 @@
         <visual>
             <geometry>
-                <cylinder radius="0.033" length="0.026"/>
+                <cylinder radius="${wheel_radius}" length="${wheel_thickness}"/>
             </geometry>
             <material name="blue"/>
@@ -89,8 +111,8 @@
         <collision>
             <geometry>
-                <sphere radius="0.033"/>
+                <sphere radius="${wheel_radius}"/>
             </geometry>
         </collision>
-        <xacro:inertial_cylinder mass="0.1" length="0.026" radius="0.033">
+        <xacro:inertial_cylinder mass="${wheel_mass}" length="${wheel_thickness}" radius="${wheel_radius}">
             <origin xyz="0 0 0" rpy="0 0 0"/>
         </xacro:inertial_cylinder>
@@ -103,10 +125,10 @@
         <parent link="chassis"/>
         <child link="caster_wheel"/>
-        <origin xyz="0.2 0 0"/>
+        <origin xyz="${caster_wheel_offset_x} 0 ${caster_wheel_offset_z}"/>
     </joint>
     <link name="caster_wheel">
         <visual>
             <geometry>
-                <sphere radius="0.033"/>
+                <sphere radius="${caster_wheel_radius}"/>
             </geometry>
             <material name="white"/>
@@ -114,8 +136,8 @@
         <collision>
             <geometry>
-                <sphere radius="0.033"/>
+                <sphere radius="${caster_wheel_radius}"/>
             </geometry>
         </collision>
-        <xacro:inertial_sphere mass="0.1" radius="0.033">
+        <xacro:inertial_sphere mass="${caster_wheel_mass}" radius="${caster_wheel_radius}">
             <origin xyz="0 0 0" rpy="0 0 0"/>
         </xacro:inertial_sphere>
@@ -126,13 +148,3 @@
         <mu2 value="0.001"/>
     </gazebo>
-    <gazebo>
-        <plugin name="gazebo_ros" filename="libgazebo_ros_init.so"/>
-    </gazebo>
-    <gazebo>
-        <plugin name="gazebo_ros_state" filename="libgazebo_ros_p3d.so">
-            <body_name>base_link</body_name>
-            <frame_name>map</frame_name>
-            <update_rate>50.0</update_rate>
-        </plugin>
-    </gazebo>
 </robot>

File: description/ros2_control.xacro (robot description, xacro)
@@ -11,5 +11,5 @@
                 <param name="baud_rate">57600</param>
                 <param name="timeout_ms">1000</param>
-                <param name="enc_counts_per_rev">3436</param>
+                <param name="enc_counts_per_rev">7260</param>
             </hardware>
             <joint name="left_wheel_joint">
@@ -56,6 +56,6 @@
     <gazebo>
         <plugin name="gazebo_ros2_control" filename="libgazebo_ros2_control.so">
-            <parameters>$(find articubot_one)/config/my_controllers.yaml</parameters>
-            <parameters>$(find articubot_one)/config/gaz_ros2_ctl_use_sim.yaml</parameters>
+            <parameters>$(find florence_bot)/config/my_controllers.yaml</parameters>
+            <parameters>$(find florence_bot)/config/gaz_ros2_ctl_use_sim.yaml</parameters>
         </plugin>
     </gazebo>
